Commit message: Add collision meshes using V-HACD

File: indy_description/robots/indy_arm.xacro (robot description, xacro)
@@ -2,5 +2,5 @@
 <robot xmlns:xacro="http://www.ros.org/wiki/xacro" name="indy">
   <!-- [ arm_id ] Namespace of the indy arm. Should be unique if multiple indy arms are used. -->
-  <!-- [ model  ] The model of the indy arm. It should be one of the folders in 'config' folder. -->
+  <!-- [ model  ] The model of the indy arm. It should be one of the folders in 'robots' folder. -->
   <xacro:macro name="indy_arm" params="arm_id:='indy' model description_pkg:='indy_description' connected_to:='' xyz:='0 0 0' rpy:='0 0 0'">
     <!-- OPTIONAL: Add a joint between the arm and the connected_to link -->

File: indy_description/robots/utils.xacro (robot description, xacro)
@@ -42,5 +42,5 @@
           <origin xyz="0 0 0" rpy="0 0 0"/>
           <geometry>
-            <mesh filename="package://${description_pkg}/meshes/${model}/collision/${model}_${link_id}.stl"/>
+            <mesh filename="package://${description_pkg}/meshes/${model}/collision/${model}_${link_id}.obj"/>
           </geometry>
         </collision>

Commit message: Add `indy_flange` link to URDF

File: indy_description/robots/indy_arm.xacro (robot description, xacro)
@@ -31,4 +31,11 @@
     <xacro:indy_joint joint_id="5"/>
     <xacro:indy_joint joint_id="6" when="${joint6_exist}"/>
+    <!-- flange -->
+    <xacro:if value="${joint6_exist}">
+      <xacro:indy_flange parent_link="${arm_id}_link7"/>
+    </xacro:if>
+    <xacro:unless value="${joint6_exist}">
+      <xacro:indy_flange parent_link="${arm_id}_link6"/>
+    </xacro:unless>
   </xacro:macro>
 </robot>

File: indy_description/robots/utils.xacro (robot description, xacro)
@@ -55,5 +55,5 @@
     </xacro:if>
   </xacro:macro>
-  <xacro:macro name="indy_joint" params="arm_id:=^ model:=^ description_pkg:=^ joint_id when:=true">
+  <xacro:macro name="indy_joint" params="arm_id:=^ model:=^ joint_id when:=true">
     <xacro:if value="${when}">
       <xacro:property name="joint_origin" value="${xacro.load_yaml(model + '/kinematics.yaml')['kinematics']['joint' + str(joint_id)]}"/>
@@ -75,3 +75,14 @@
     </xacro:if>
   </xacro:macro>
+  <xacro:macro name="indy_flange" params="arm_id:=^ model:=^ parent_link">
+    <link name="${arm_id}_flange"/>
+    <xacro:property name="joint_origin" value="${xacro.load_yaml(model + '/kinematics.yaml')['kinematics']['flange']}"/>
+    <joint name="${arm_id}_joint_flange" type="fixed">
+      <parent link="${parent_link}"/>
+      <child link="${arm_id}_flange"/>
+      <origin
+        xyz="${joint_origin['x']} ${joint_origin['y']} ${joint_origin['z']}"
+        rpy="${joint_origin['roll']} ${joint_origin['pitch']} ${joint_origin['yaw']}"/>
+    </joint>
+  </xacro:macro>
 </robot>

Commit message: Feat: change indy_flange to indy_flange_nrmkapi

File: indy_description/robots/indy_arm.xacro (robot description, xacro)
@@ -33,8 +33,8 @@
     <!-- flange -->
     <xacro:if value="${joint6_exist}">
-      <xacro:indy_flange parent_link="${arm_id}_link7"/>
+      <xacro:indy_flange_nrmkapi parent_link="${arm_id}_link7"/>
     </xacro:if>
     <xacro:unless value="${joint6_exist}">
-      <xacro:indy_flange parent_link="${arm_id}_link6"/>
+      <xacro:indy_flange_nrmkapi parent_link="${arm_id}_link6"/>
     </xacro:unless>
   </xacro:macro>

File: indy_description/robots/utils.xacro (robot description, xacro)
@@ -75,10 +75,10 @@
     </xacro:if>
   </xacro:macro>
-  <xacro:macro name="indy_flange" params="arm_id:=^ model:=^ parent_link">
-    <link name="${arm_id}_flange"/>
+  <xacro:macro name="indy_flange_nrmkapi" params="arm_id:=^ model:=^ parent_link">
+    <link name="${arm_id}_flange_nrmkapi"/>
     <xacro:property name="joint_origin" value="${xacro.load_yaml(model + '/kinematics.yaml')['kinematics']['flange']}"/>
     <joint name="${arm_id}_joint_flange" type="fixed">
       <parent link="${parent_link}"/>
-      <child link="${arm_id}_flange"/>
+      <child link="${arm_id}_flange_nrmkapi"/>
       <origin
         xyz="${joint_origin['x']} ${joint_origin['y']} ${joint_origin['z']}"

Commit message: Add indy_flange_nrmkapi (from IndyDCP) and correct URDFs

File: indy_description/robots/indy_arm.xacro (robot description, xacro)
@@ -33,8 +33,8 @@
     <!-- flange -->
     <xacro:if value="${joint6_exist}">
-      <xacro:indy_flange_nrmkapi parent_link="${arm_id}_link7"/>
+      <xacro:indy_flange parent_link="${arm_id}_link7"/>
     </xacro:if>
     <xacro:unless value="${joint6_exist}">
-      <xacro:indy_flange_nrmkapi parent_link="${arm_id}_link6"/>
+      <xacro:indy_flange parent_link="${arm_id}_link6"/>
     </xacro:unless>
   </xacro:macro>

File: indy_description/robots/utils.xacro (robot description, xacro)
@@ -75,10 +75,10 @@
     </xacro:if>
   </xacro:macro>
-  <xacro:macro name="indy_flange_nrmkapi" params="arm_id:=^ model:=^ parent_link">
-    <link name="${arm_id}_flange_nrmkapi"/>
+  <xacro:macro name="indy_flange" params="arm_id:=^ model:=^ parent_link">
+    <link name="${arm_id}_flange"/>
     <xacro:property name="joint_origin" value="${xacro.load_yaml(model + '/kinematics.yaml')['kinematics']['flange']}"/>
     <joint name="${arm_id}_joint_flange" type="fixed">
       <parent link="${parent_link}"/>
-      <child link="${arm_id}_flange_nrmkapi"/>
+      <child link="${arm_id}_flange"/>
       <origin
         xyz="${joint_origin['x']} ${joint_origin['y']} ${joint_origin['z']}"
