Commit message: add use_hand argument for visuzlaize

File: indy_description/robots/indy_arm.urdf.xacro (robot description, xacro)
@@ -7,8 +7,25 @@
   <xacro:arg name="use_fake_hardware" default="true"/>
   <xacro:arg name="fake_sensor_commands" default="true"/>
+  <xacro:arg name="use_hand" default="false"/>
   <!-- Include the model -->
   <!-- <xacro:include filename="$(find indy_description)/robots/test.xacro"/> -->
   <xacro:include filename="$(find indy_description)/robots/indy_arm.xacro"/>
   <xacro:indy_arm arm_id="$(arg arm_id)" model="$(arg model)" connected_to="$(arg connected_to)"/>
+  <xacro:if value="$(arg use_hand)">
+    <xacro:include filename="$(find amm_hand_v2_description)/urdf/hand_v2_0_macro.xacro"/>
+    <xacro:hand_v2_0
+      prefix=""
+      joint_limits="${xacro.load_yaml('$(find amm_hand_v2_description)/urdf/joint_limits.yaml')}"
+      inertials="${xacro.load_yaml('$(find amm_hand_v2_description)/urdf/inertials.yaml')}"
+      simplified="false"
+      isaac_gym="false"
+      palm_is_base="false"
+    />
+    <joint name="hand_mount" type="fixed">
+      <parent link="indy_flange"/>
+      <child  link="hand_base"/>
+      <origin xyz="0 0 0" rpy="0 0 0"/>
+    </joint>
+</xacro:if>
   <!-- Include the ros2_control plugin -->
   <xacro:include filename="$(find indy_description)/robots/indy_arm.ros2_control.xacro"/>

Commit message: rotate hand base

File: indy_description/robots/indy_arm.urdf.xacro (robot description, xacro)
@@ -25,5 +25,5 @@
       <parent link="indy_flange"/>
       <child  link="hand_base"/>
-      <origin xyz="0 0 0" rpy="0 0 0"/>
+      <origin xyz="0 0 0" rpy="0 0 -${pi/2}"/>
     </joint>
 </xacro:if>

Commit message: nsquare settings

File: indy_description/robots/indy_arm.urdf.xacro (robot description, xacro)
@@ -25,5 +25,5 @@
       <parent link="indy_flange"/>
       <child  link="hand_base"/>
-      <origin xyz="0 0 0" rpy="0 0 -${pi/2}"/>
+      <origin xyz="0 0 0" rpy="0 0 ${pi/2}"/>
     </joint>
 </xacro:if>

Commit message: 5g demo settings

File: indy_description/robots/indy_arm.urdf.xacro (robot description, xacro)
@@ -25,5 +25,6 @@
       <parent link="indy_flange"/>
       <child  link="hand_base"/>
-      <origin xyz="0 0 0" rpy="0 0 ${pi/2}"/>
+      <origin xyz="0 0 0.06" rpy="0 0 ${-pi/2}"/>
+      <!-- <origin xyz="0 0 0.06" rpy="0 0 ${pi/2}"/> -->
     </joint>
 </xacro:if>

Commit message: change joint limits for moveit

File: indy_description/robots/indy_arm.urdf.xacro (robot description, xacro)
@@ -25,6 +25,6 @@
       <parent link="indy_flange"/>
       <child  link="hand_base"/>
-      <origin xyz="0 0 0.06" rpy="0 0 ${-pi/2}"/>
-      <!-- <origin xyz="0 0 0.06" rpy="0 0 ${pi/2}"/> -->
+      <!-- <origin xyz="0 0 0.06" rpy="0 0 ${-pi/2}"/> -->
+      <origin xyz="0 0 0.06" rpy="0 0 ${pi/2}"/>
     </joint>
 </xacro:if>

File: indy_moveit_config/srdf/group_definition.xacro (robot description, xacro)
@@ -12,5 +12,5 @@
       <joint name="${arm_id}_joint4" value="0"/>
       <joint name="${arm_id}_joint5" value="${-pi/2}"/>
-      <joint name="${arm_id}_joint6" value="0"/>
+      <!-- <joint name="${arm_id}_joint6" value="0"/> -->
       <joint name="${arm_id}_flange" value="0"/>
     </group_state>

File: indy_moveit_config/srdf/indy_arm.xacro (robot description, xacro)
@@ -24,6 +24,6 @@
     <disable_collisions link1="${arm_id}_link5" link2="${arm_id}_link6" reason="Adjacent"/>
     <disable_collisions link1="${arm_id}_link6" link2="${arm_id}_link7" reason="Adjacent"/>
-    <disable_collisions link1="${arm_id}_link7" link2="${arm_id}_flange" reason="Adjacent"/>
-    <disable_collisions link1="${arm_id}_link7" link2="${arm_id}_flange" reason="Default"/>
+    <!-- <disable_collisions link1="${arm_id}_link7" link2="${arm_id}_flange" reason="Adjacent"/>
+    <disable_collisions link1="${arm_id}_link7" link2="${arm_id}_flange" reason="Default"/> -->
   </xacro:macro>
 </robot>
