Commit message: Change collision mesh from obj to binary stl

File: indy_description/robots/utils.xacro (robot description, xacro)
@@ -44,5 +44,6 @@
           <origin xyz="0 0 0" rpy="0 0 0"/>
           <geometry>
-            <mesh filename="package://${description_pkg}/meshes/${model}/collision/${model}_${link_id}.obj"/>
+            <!-- <mesh filename="package://${description_pkg}/meshes/${model}/collision/${model}_${link_id}.obj"/> -->
+            <mesh filename="package://${description_pkg}/meshes/${model}/collision/${model}_${link_id}.stl"/>
           </geometry>
         </collision>

Commit message: Fix a bug in urdf (load yaml path error when include xacro in other pkgs)

File: indy_description/robots/utils.xacro (robot description, xacro)
@@ -11,5 +11,5 @@
   <!-- ========================================================== -->
   <xacro:macro name="set_property_if_joint_exist" params="joint_id property_name">
-    <xacro:property name="kinematics_dict" value="${xacro.load_yaml(model + '/kinematics.yaml')['kinematics']}"/>
+    <xacro:property name="kinematics_dict" value="${xacro.load_yaml('$(find indy_description)/robots/$(arg model)/kinematics.yaml')['kinematics']}"/>
     <xacro:property name="key" value="joint${joint_id}"/>
     <xacro:if value="${key in kinematics_dict}">
@@ -28,5 +28,5 @@
   <xacro:macro name="indy_link" params="arm_id:=^ model:=^ description_pkg:=^ link_id color when:=true">
     <xacro:if value="${when}">
-      <xacro:property name="physical_parameters" value="${xacro.load_yaml(model + '/physical_parameters.yaml')['inertia_parameters']}"/>
+      <xacro:property name="physical_parameters" value="${xacro.load_yaml('$(find indy_description)/robots/$(arg model)/physical_parameters.yaml')['inertia_parameters']}"/>
       <xacro:property name="link_mass" value="${physical_parameters['link' + str(link_id) + '_mass']}"/>
       <xacro:property name="link_inertia" value="${physical_parameters['link' + str(link_id)]}"/>
@@ -57,6 +57,6 @@
   <xacro:macro name="indy_joint" params="arm_id:=^ model:=^ joint_id when:=true">
     <xacro:if value="${when}">
-      <xacro:property name="joint_origin" value="${xacro.load_yaml(model + '/kinematics.yaml')['kinematics']['joint' + str(joint_id)]}"/>
-      <xacro:property name="joint_limit" value="${xacro.load_yaml(model + '/joint_limits.yaml')['joint_limits']['joint' + str(joint_id)]}"/>
+      <xacro:property name="joint_origin" value="${xacro.load_yaml('$(find indy_description)/robots/$(arg model)/kinematics.yaml')['kinematics']['joint' + str(joint_id)]}"/>
+      <xacro:property name="joint_limit" value="${xacro.load_yaml('$(find indy_description)/robots/$(arg model)/joint_limits.yaml')['joint_limits']['joint' + str(joint_id)]}"/>
       <joint name="${arm_id}_joint${joint_id}" type="revolute">
         <parent link="${arm_id}_link${joint_id}"/>
@@ -77,5 +77,5 @@
   <xacro:macro name="indy_flange" params="arm_id:=^ model:=^ parent_link">
     <link name="${arm_id}_flange"/>
-    <xacro:property name="joint_origin" value="${xacro.load_yaml(model + '/kinematics.yaml')['kinematics']['flange']}"/>
+    <xacro:property name="joint_origin" value="${xacro.load_yaml('$(find indy_description)/robots/$(arg model)/kinematics.yaml')['kinematics']['flange']}"/>
     <joint name="${arm_id}_joint_flange" type="fixed">
       <parent link="${parent_link}"/>

Commit message: Add 'joint6_exist' macro to remove joint7 warnings

File: indy_description/robots/utils.xacro (robot description, xacro)
@@ -10,6 +10,7 @@
   <!-- Function definitions                                       -->
   <!-- ========================================================== -->
-  <xacro:macro name="set_property_if_joint_exist" params="joint_id property_name">
-    <xacro:property name="kinematics_dict" value="${xacro.load_yaml(model + '/kinematics.yaml')['kinematics']}"/>
+  <xacro:macro name="set_property_if_joint_exist" params="joint_id property_name model:=^ description_pkg:=^">
+    <xacro:property name="_desc" value="$(find ${description_pkg})"/>
+    <xacro:property name="kinematics_dict" value="${xacro.load_yaml(_desc + '/robots/' + model + '/kinematics.yaml')['kinematics']}"/>
     <xacro:property name="key" value="joint${joint_id}"/>
     <xacro:if value="${key in kinematics_dict}">

File: indy_moveit_config/srdf/group_definition.xacro (robot description, xacro)
@@ -1,5 +1,5 @@
 <?xml version="1.0" encoding="UTF-8"?>
 <robot xmlns:xacro="http://www.ros.org/wiki/xacro" name="indy">
-  <xacro:macro name="group_definition" params="group_name arm_id tip_link">
+  <xacro:macro name="group_definition" params="group_name arm_id tip_link description_pkg:='indy_description' model:='indy7'">
     <group name="${group_name}">
       <chain base_link="${arm_id}_link0" tip_link="${tip_link}"/>
@@ -13,5 +13,10 @@
       <joint name="${arm_id}_joint5" value="${-pi/2}"/>
       <!-- <joint name="${arm_id}_joint6" value="0"/> -->
-      <joint name="${arm_id}_flange" value="0"/>
+      <!-- <joint name="${arm_id}_flange" value="0"/> -->
+    <xacro:include filename="$(find ${description_pkg})/robots/utils.xacro"/>
+    <xacro:set_property_if_joint_exist joint_id="6" property_name="joint6_exist"/>
+    <xacro:if value="${joint6_exist}">
+      <joint name="${arm_id}_joint6" value="0"/>
+    </xacro:if>
     </group_state>
   </xacro:macro>

File: indy_moveit_config/srdf/indy_arm.srdf.xacro (robot description, xacro)
@@ -2,6 +2,8 @@
 <robot xmlns:xacro="http://www.ros.org/wiki/xacro" name="indy">
   <xacro:arg name="arm_id" default="indy"/> <!-- Name of this indy -->
+  <xacro:arg name="model" default="indy7"/> <!-- Model of the indy arm -->
   <xacro:property name="arm_id" value="$(arg arm_id)"/>
+  <xacro:property name="model" value="$(arg model)"/>
   <xacro:include filename="$(find indy_moveit_config)/srdf/indy_arm.xacro"/>
-  <xacro:indy_arm arm_id="${arm_id}"/>
+  <xacro:indy_arm arm_id="${arm_id}" model="${model}"/>
 </robot>

File: indy_moveit_config/srdf/indy_arm.xacro (robot description, xacro)
@@ -1,5 +1,5 @@
 <?xml version="1.0" ?>
 <robot xmlns:xacro="http://www.ros.org/wiki/xacro" name="indy">
-  <xacro:macro name="indy_arm" params="arm_id:='indy' ">
+  <xacro:macro name="indy_arm" params="arm_id:='indy' description_pkg:='indy_description' model:='indy7'">
     <xacro:include filename="$(find indy_moveit_config)/srdf/group_definition.xacro"/>
     <xacro:group_definition arm_id="${arm_id}" group_name="${arm_id}_arm" tip_link="${arm_id}_flange"/>
@@ -23,7 +23,16 @@
     <disable_collisions link1="${arm_id}_link4" link2="${arm_id}_flange" reason="Never"/>
     <disable_collisions link1="${arm_id}_link5" link2="${arm_id}_link6" reason="Adjacent"/>
-    <disable_collisions link1="${arm_id}_link6" link2="${arm_id}_link7" reason="Adjacent"/>
-    <!-- <disable_collisions link1="${arm_id}_link7" link2="${arm_id}_flange" reason="Adjacent"/>
-    <disable_collisions link1="${arm_id}_link7" link2="${arm_id}_flange" reason="Default"/> -->
+    <!-- <disable_collisions link1="${arm_id}_link6" link2="${arm_id}_link7" reason="Adjacent"/> -->
+    <!-- <disable_collisions link1="${arm_id}_link7" link2="${arm_id}_flange" reason="Adjacent"/> -->
+    <xacro:include filename="$(find ${description_pkg})/robots/utils.xacro"/>
+    <xacro:set_property_if_joint_exist joint_id="6" property_name="joint6_exist"/>
+    <xacro:if value="${joint6_exist}">
+      <disable_collisions link1="${arm_id}_link6" link2="${arm_id}_link7" reason="Adjacent"/>
+      <disable_collisions link1="${arm_id}_link6" link2="${arm_id}_flange" reason="Never"/>
+      <disable_collisions link1="${arm_id}_link7" link2="${arm_id}_flange" reason="Adjacent"/>
+    </xacro:if>
+    <xacro:unless value="${joint6_exist}">
+      <disable_collisions link1="${arm_id}_link6" link2="${arm_id}_flange" reason="Adjacent"/>
+    </xacro:unless>
   </xacro:macro>
 </robot>
