Commit message: Add indy_sim_gazebo package (w/o control)

File: indy_description/robots/indy_arm.ros2_control.xacro (robot description, xacro)
@@ -1,20 +1,33 @@
 <?xml version="1.0" encoding="UTF-8"?>
 <robot xmlns:xacro="http://www.ros.org/wiki/xacro">
-  <xacro:macro name="indy_arm_ros2_control" params="ns model description_pkg:='indy_description'  use_fake_hardware:=^|false fake_sensor_commands:=^|false">
+  <xacro:macro
+    name="indy_arm_ros2_control"
+    params="ns
+            model
+            description_pkg:='indy_description'
+            target_system:='fake_hardware'
+            fake_sensor_commands:=^|false">
     <ros2_control name="IndyHardwareInterface" type="system">
       <hardware>
-        <xacro:if value="${use_fake_hardware}">
+        <xacro:if value="${target_system == 'real_hardware'}">
+          <!-- TODO indy_hardware plugin is not yet implemented -->
+          <!-- <plugin>indy_hardware/IndyHardwareInterface</plugin> -->
+        </xacro:if>
+        <xacro:if value="${target_system == 'fake_hardware'}">
           <plugin>fake_components/GenericSystem</plugin>
           <param name="fake_sensor_commands">${fake_sensor_commands}</param>
           <param name="state_following_offset">0.0</param>
         </xacro:if>
-        <xacro:unless value="${use_fake_hardware}">
-          <!-- TODO indy_hardware plugin is not yet implemented -->
-          <!-- <plugin>indy_hardware/IndyHardwareInterface</plugin> -->
-        </xacro:unless>
+        <xacro:if value="${target_system == 'gazebo'}">
+          <plugin>gz_ros2_control/GazeboSimSystem</plugin>
+        </xacro:if>
+        <xacro:if value="${target_system not in ['real_hardware', 'fake_hardware', 'gazebo']}">
+          <xacro:error text="Unknown target system: '${target_system}'"/>
+        </xacro:if>
       </hardware>
-      <xacro:macro name="configure_joint" params="ns:=^ model:=^ joint_id initial_position when:=true">
+      <xacro:macro name="configure_joint" params="ns:=^ model:=^ description_pkg:=^ joint_id initial_position when:=true">
         <xacro:if value="${when}">
-          <xacro:property name="joint_limit" value="${xacro.load_yaml(model + '/joint_limits.yaml')['joint_limits']['joint' + str(joint_id)]}"/>
+          <xacro:property name="config_dir" value="$(find ${description_pkg})/robots/${model}"/>
+          <xacro:property name="joint_limit" value="${xacro.load_yaml(config_dir + '/joint_limits.yaml')['joint_limits']['joint' + str(joint_id)]}"/>
           <joint name="${ns}_joint${joint_id}">
             <param name="initial_position">${initial_position}</param>

File: indy_description/robots/indy_arm.urdf.xacro (robot description, xacro)
@@ -5,12 +5,21 @@
   <xacro:arg name="model" default="indy7"/>    <!-- Model of the indy arm -->
   <xacro:arg name="connected_to" default=""/>  <!-- Link to which the indy arm is connected to -->
-  <xacro:arg name="use_fake_hardware" default="true"/>
+  <!-- ROS2 control parameters
+  Available target systems are
+    - real_hardware
+    - fake_hardware
+    - gazebo (for Gazebo Fortress or later)
+  -->
+  <xacro:arg name="target_system" default="fake_hardware"/>
   <xacro:arg name="fake_sensor_commands" default="true"/>
   <!-- Include the model -->
-  <!-- <xacro:include filename="$(find indy_description)/robots/test.xacro"/> -->
   <xacro:include filename="$(find indy_description)/robots/indy_arm.xacro"/>
   <xacro:indy_arm arm_id="$(arg arm_id)" model="$(arg model)" connected_to="$(arg connected_to)"/>
   <!-- Include the ros2_control plugin -->
   <xacro:include filename="$(find indy_description)/robots/indy_arm.ros2_control.xacro"/>
-  <xacro:indy_arm_ros2_control ns="$(arg arm_id)" model="$(arg model)" use_fake_hardware="$(arg use_fake_hardware)" fake_sensor_commands="$(arg fake_sensor_commands)"/>
+  <xacro:indy_arm_ros2_control
+    ns="$(arg arm_id)"
+    model="$(arg model)"
+    target_system="$(arg target_system)"
+    fake_sensor_commands="$(arg fake_sensor_commands)"/>
 </robot>

File: indy_description/robots/utils.xacro (robot description, xacro)
@@ -10,6 +10,7 @@
   <!-- Function definitions                                       -->
   <!-- ========================================================== -->
-  <xacro:macro name="set_property_if_joint_exist" params="joint_id property_name">
-    <xacro:property name="kinematics_dict" value="${xacro.load_yaml(model + '/kinematics.yaml')['kinematics']}"/>
+  <xacro:macro name="set_property_if_joint_exist" params="description_pkg:=^ joint_id property_name">
+    <xacro:property name="config_dir" value="$(find ${description_pkg})/robots/${model}"/>
+    <xacro:property name="kinematics_dict" value="${xacro.load_yaml(config_dir + '/kinematics.yaml')['kinematics']}"/>
     <xacro:property name="key" value="joint${joint_id}"/>
     <xacro:if value="${key in kinematics_dict}">
@@ -28,5 +29,6 @@
   <xacro:macro name="indy_link" params="arm_id:=^ model:=^ description_pkg:=^ link_id color when:=true">
     <xacro:if value="${when}">
-      <xacro:property name="physical_parameters" value="${xacro.load_yaml(model + '/physical_parameters.yaml')['inertia_parameters']}"/>
+      <xacro:property name="config_dir" value="$(find ${description_pkg})/robots/${model}"/>
+      <xacro:property name="physical_parameters" value="${xacro.load_yaml(config_dir + '/physical_parameters.yaml')['inertia_parameters']}"/>
       <xacro:property name="link_mass" value="${physical_parameters['link' + str(link_id) + '_mass']}"/>
       <xacro:property name="link_inertia" value="${physical_parameters['link' + str(link_id)]}"/>
@@ -57,6 +59,7 @@
   <xacro:macro name="indy_joint" params="arm_id:=^ model:=^ description_pkg:=^ joint_id when:=true">
     <xacro:if value="${when}">
-      <xacro:property name="joint_origin" value="${xacro.load_yaml(model + '/kinematics.yaml')['kinematics']['joint' + str(joint_id)]}"/>
-      <xacro:property name="joint_limit" value="${xacro.load_yaml(model + '/joint_limits.yaml')['joint_limits']['joint' + str(joint_id)]}"/>
+      <xacro:property name="config_dir" value="$(find ${description_pkg})/robots/${model}"/>
+      <xacro:property name="joint_origin" value="${xacro.load_yaml(config_dir + '/kinematics.yaml')['kinematics']['joint' + str(joint_id)]}"/>
+      <xacro:property name="joint_limit" value="${xacro.load_yaml(config_dir + '/joint_limits.yaml')['joint_limits']['joint' + str(joint_id)]}"/>
       <joint name="${arm_id}_joint${joint_id}" type="revolute">
         <parent link="${arm_id}_link${joint_id}"/>

Commit message: Add a missing description_pkg dir

File: indy_description/robots/indy_arm.ros2_control.xacro (robot description, xacro)
@@ -14,7 +14,8 @@
         </xacro:unless>
       </hardware>
-      <xacro:macro name="configure_joint" params="ns:=^ model:=^ joint_id initial_position when:=true">
+      <xacro:macro name="configure_joint" params="ns:=^ model:=^ description_pkg:=^ joint_id initial_position when:=true">
         <xacro:if value="${when}">
-          <xacro:property name="joint_limit" value="${xacro.load_yaml(model + '/joint_limits.yaml')['joint_limits']['joint' + str(joint_id)]}"/>
+          <xacro:property name="_desc" value="$(find ${description_pkg})"/>
+          <xacro:property name="joint_limit" value="${xacro.load_yaml(_desc + '/robots/' + model + '/joint_limits.yaml')['joint_limits']['joint' + str(joint_id)]}"/>
           <joint name="${ns}_joint${joint_id}">
             <param name="initial_position">${initial_position}</param>

File: indy_description/robots/utils.xacro (robot description, xacro)
@@ -29,5 +29,6 @@
   <xacro:macro name="indy_link" params="arm_id:=^ model:=^ description_pkg:=^ link_id color when:=true">
     <xacro:if value="${when}">
-      <xacro:property name="physical_parameters" value="${xacro.load_yaml(model + '/physical_parameters.yaml')['inertia_parameters']}"/>
+      <xacro:property name="_desc" value="$(find ${description_pkg})"/>
+      <xacro:property name="physical_parameters" value="${xacro.load_yaml(_desc + '/robots/' + model + '/physical_parameters.yaml')['inertia_parameters']}"/>
       <xacro:property name="link_mass" value="${physical_parameters['link' + str(link_id) + '_mass']}"/>
       <xacro:property name="link_inertia" value="${physical_parameters['link' + str(link_id)]}"/>
@@ -56,8 +57,9 @@
     </xacro:if>
   </xacro:macro>
-  <xacro:macro name="indy_joint" params="arm_id:=^ model:=^ joint_id when:=true">
+  <xacro:macro name="indy_joint" params="arm_id:=^ model:=^ description_pkg:=^ joint_id when:=true">
     <xacro:if value="${when}">
-      <xacro:property name="joint_origin" value="${xacro.load_yaml(model + '/kinematics.yaml')['kinematics']['joint' + str(joint_id)]}"/>
-      <xacro:property name="joint_limit" value="${xacro.load_yaml(model + '/joint_limits.yaml')['joint_limits']['joint' + str(joint_id)]}"/>
+      <xacro:property name="_desc" value="$(find ${description_pkg})"/>
+      <xacro:property name="joint_origin" value="${xacro.load_yaml(_desc + '/robots/' + model + '/kinematics.yaml')['kinematics']['joint' + str(joint_id)]}"/>
+      <xacro:property name="joint_limit" value="${xacro.load_yaml(_desc + '/robots/' + model + '/joint_limits.yaml')['joint_limits']['joint' + str(joint_id)]}"/>
       <joint name="${arm_id}_joint${joint_id}" type="revolute">
         <parent link="${arm_id}_link${joint_id}"/>
@@ -76,7 +78,8 @@
     </xacro:if>
   </xacro:macro>
-  <xacro:macro name="indy_flange" params="arm_id:=^ model:=^ parent_link">
+  <xacro:macro name="indy_flange" params="arm_id:=^ model:=^ description_pkg:=^ parent_link">
     <link name="${arm_id}_flange"/>
-    <xacro:property name="joint_origin" value="${xacro.load_yaml(model + '/kinematics.yaml')['kinematics']['flange']}"/>
+    <xacro:property name="_desc" value="$(find ${description_pkg})"/>
+    <xacro:property name="joint_origin" value="${xacro.load_yaml(_desc + '/robots/' + model + '/kinematics.yaml')['kinematics']['flange']}"/>
     <joint name="${arm_id}_joint_flange" type="fixed">
       <parent link="${parent_link}"/>
