Commit message: WIP: add indy_arm_hand planning group

File: indy_moveit_config/srdf/indy_arm.srdf.xacro (robot description, xacro)
@@ -3,7 +3,9 @@
   <xacro:arg name="arm_id" default="indy"/> <!-- Name of this indy -->
   <xacro:arg name="dof" default="7"/> <!-- Number of degrees of freedom -->
+  <xacro:arg name="hand" default="false"/> <!-- Whether the hand is attached -->
   <xacro:property name="arm_id" value="$(arg arm_id)"/>
   <xacro:property name="dof" value="$(arg dof)"/>
+  <xacro:property name="hand" value="$(arg hand)"/>
   <xacro:include filename="$(find indy_moveit_config)/srdf/indy_arm.xacro"/>
-  <xacro:indy_arm arm_id="${arm_id}" dof="${dof}"/>
+  <xacro:indy_arm arm_id="${arm_id}" dof="${dof}" hand="${hand}"/>
 </robot>

File: indy_moveit_config/srdf/indy_arm.xacro (robot description, xacro)
@@ -1,7 +1,10 @@
 <?xml version="1.0" ?>
 <robot xmlns:xacro="http://www.ros.org/wiki/xacro" name="indy">
-  <xacro:macro name="indy_arm" params="arm_id:='indy' dof:='7'">
+  <xacro:macro name="indy_arm" params="arm_id:='indy' dof:='7' hand:='false'">
     <xacro:include filename="$(find indy_moveit_config)/srdf/group_definition.xacro"/>
     <xacro:group_definition arm_id="${arm_id}" group_name="${arm_id}_arm" tip_link="${arm_id}_flange" dof="${dof}"/>
+    <xacro:if value="${hand}">
+        <xacro:group_definition arm_id="${arm_id}" group_name="${arm_id}_arm_hand" tip_link="hand_palm" dof="${dof}"/>
+    </xacro:if>
     <virtual_joint name="virtual_joint" type="fixed" parent_frame="world" child_link="${arm_id}_link0"/>
     <disable_collisions link1="${arm_id}_link0" link2="${arm_id}_link1" reason="Adjacent"/>
