Commit message: Fix the Indy DoF problem (now, you can choose 6dof or 7dof.)

File: indy_moveit_config/srdf/group_definition.xacro (robot description, xacro)
@@ -1,17 +1,37 @@
 <?xml version="1.0" encoding="UTF-8"?>
 <robot xmlns:xacro="http://www.ros.org/wiki/xacro" name="indy">
-  <xacro:macro name="group_definition" params="group_name arm_id tip_link">
+  <xacro:macro name="group_definition" params="group_name arm_id tip_link dof:='7'">
     <group name="${group_name}">
       <chain base_link="${arm_id}_link0" tip_link="${tip_link}"/>
     </group>
-    <group_state name="ready" group="${group_name}">
+    <group_state name="home" group="${group_name}">
       <joint name="${arm_id}_joint0" value="0"/>
       <joint name="${arm_id}_joint1" value="0"/>
       <joint name="${arm_id}_joint2" value="0"/>
-      <joint name="${arm_id}_joint3" value="${-pi/2}"/>
+      <joint name="${arm_id}_joint3" value="0"/>
       <joint name="${arm_id}_joint4" value="0"/>
-      <joint name="${arm_id}_joint5" value="${-pi/2}"/>
-      <!-- <joint name="${arm_id}_joint6" value="0"/>
-      <joint name="${arm_id}_flange" value="0"/> -->
+      <joint name="${arm_id}_joint5" value="0"/>
+      <xacro:if value="${dof == 7}">
+        <joint name="${arm_id}_joint6" value="0"/>
+      </xacro:if>
+    </group_state>
+    <group_state name="ready" group="${group_name}">
+      <xacro:if value="${dof == 7}">
+        <joint name="${arm_id}_joint0" value="0"/>
+        <joint name="${arm_id}_joint1" value="0"/>
+        <joint name="${arm_id}_joint2" value="0"/>
+        <joint name="${arm_id}_joint3" value="${-pi/2}"/>
+        <joint name="${arm_id}_joint4" value="0"/>
+        <joint name="${arm_id}_joint5" value="${-pi/2}"/>
+        <joint name="${arm_id}_joint6" value="0"/>
+      </xacro:if>
+      <xacro:unless value="${dof == 7}">
+        <joint name="${arm_id}_joint0" value="0"/>
+        <joint name="${arm_id}_joint1" value="0"/>
+        <joint name="${arm_id}_joint2" value="${-pi/2}"/>
+        <joint name="${arm_id}_joint3" value="0"/>
+        <joint name="${arm_id}_joint4" value="${-pi/2}"/>
+        <joint name="${arm_id}_joint5" value="0"/>
+      </xacro:unless>
     </group_state>
   </xacro:macro>

File: indy_moveit_config/srdf/indy_arm.srdf.xacro (robot description, xacro)
@@ -2,6 +2,8 @@
 <robot xmlns:xacro="http://www.ros.org/wiki/xacro" name="indy">
   <xacro:arg name="arm_id" default="indy"/> <!-- Name of this indy -->
+  <xacro:arg name="dof" default="7"/> <!-- Number of degrees of freedom -->
   <xacro:property name="arm_id" value="$(arg arm_id)"/>
+  <xacro:property name="dof" value="$(arg dof)"/>
   <xacro:include filename="$(find indy_moveit_config)/srdf/indy_arm.xacro"/>
-  <xacro:indy_arm arm_id="${arm_id}"/>
+  <xacro:indy_arm arm_id="${arm_id}" dof="${dof}"/>
 </robot>

File: indy_moveit_config/srdf/indy_arm.xacro (robot description, xacro)
@@ -1,7 +1,7 @@
 <?xml version="1.0" ?>
 <robot xmlns:xacro="http://www.ros.org/wiki/xacro" name="indy">
-  <xacro:macro name="indy_arm" params="arm_id:='indy' ">
+  <xacro:macro name="indy_arm" params="arm_id:='indy' dof:='7'">
     <xacro:include filename="$(find indy_moveit_config)/srdf/group_definition.xacro"/>
-    <xacro:group_definition arm_id="${arm_id}" group_name="${arm_id}_arm" tip_link="${arm_id}_flange"/>
+    <xacro:group_definition arm_id="${arm_id}" group_name="${arm_id}_arm" tip_link="${arm_id}_flange" dof="${dof}"/>
     <virtual_joint name="virtual_joint" type="fixed" parent_frame="world" child_link="${arm_id}_link0"/>
     <disable_collisions link1="${arm_id}_link0" link2="${arm_id}_link1" reason="Adjacent"/>
@@ -17,12 +17,19 @@
     <disable_collisions link1="${arm_id}_link3" link2="${arm_id}_link4" reason="Adjacent"/>
     <disable_collisions link1="${arm_id}_link3" link2="${arm_id}_link5" reason="Never"/>
+    <disable_collisions link1="${arm_id}_link3" link2="${arm_id}_flange" reason="Never"/>
     <disable_collisions link1="${arm_id}_link3" link2="${arm_id}_link6" reason="Never"/>
-    <disable_collisions link1="${arm_id}_link3" link2="${arm_id}_flange" reason="Never"/>
     <disable_collisions link1="${arm_id}_link4" link2="${arm_id}_link5" reason="Adjacent"/>
+    <disable_collisions link1="${arm_id}_link4" link2="${arm_id}_flange" reason="Never"/>
     <disable_collisions link1="${arm_id}_link4" link2="${arm_id}_link6" reason="Never"/>
-    <disable_collisions link1="${arm_id}_link4" link2="${arm_id}_flange" reason="Never"/>
     <disable_collisions link1="${arm_id}_link5" link2="${arm_id}_link6" reason="Adjacent"/>
     <disable_collisions link1="${arm_id}_link6" link2="${arm_id}_flange" reason="Adjacent"/>
     <disable_collisions link1="${arm_id}_link6" link2="${arm_id}_flange" reason="Default"/>
+    <disable_collisions link1="${arm_id}_link6" link2="${arm_id}_flange" reason="Default"/>
+    <xacro:if value="${dof == 7}">
+      <disable_collisions link1="${arm_id}_link7" link2="${arm_id}_link4" reason="Never"/>
+      <disable_collisions link1="${arm_id}_link7" link2="${arm_id}_link5" reason="Never"/>
+      <disable_collisions link1="${arm_id}_link7" link2="${arm_id}_link6" reason="Adjacent"/>
+      <disable_collisions link1="${arm_id}_link7" link2="${arm_id}_flange" reason="Default"/>
+    </xacro:if>
   </xacro:macro>
 </robot>

Commit message: modify urdf for moveit planning

File: indy_moveit_config/srdf/group_definition.xacro (robot description, xacro)
@@ -12,6 +12,6 @@
       <joint name="${arm_id}_joint4" value="0"/>
       <joint name="${arm_id}_joint5" value="${-pi/2}"/>
-      <!-- <joint name="${arm_id}_joint6" value="0"/>
-      <joint name="${arm_id}_flange" value="0"/> -->
+      <joint name="${arm_id}_joint6" value="0"/>
+      <joint name="${arm_id}_flange" value="0"/>
     </group_state>
   </xacro:macro>

File: indy_moveit_config/srdf/indy_arm.xacro (robot description, xacro)
@@ -23,6 +23,7 @@
     <disable_collisions link1="${arm_id}_link4" link2="${arm_id}_flange" reason="Never"/>
     <disable_collisions link1="${arm_id}_link5" link2="${arm_id}_link6" reason="Adjacent"/>
-    <disable_collisions link1="${arm_id}_link6" link2="${arm_id}_flange" reason="Adjacent"/>
-    <disable_collisions link1="${arm_id}_link6" link2="${arm_id}_flange" reason="Default"/>
+    <disable_collisions link1="${arm_id}_link6" link2="${arm_id}_link7" reason="Adjacent"/>
+    <disable_collisions link1="${arm_id}_link7" link2="${arm_id}_flange" reason="Adjacent"/>
+    <disable_collisions link1="${arm_id}_link7" link2="${arm_id}_flange" reason="Default"/>
   </xacro:macro>
 </robot>
